Commit message: feat: 统一设备工作流、任务采集与策略客户端

File: src/robots/zoo/dual_yam/assets/yam.urdf (robot description, URDF)
Before this commit: robot yam_fallback, 9 links, 8 joints
Links:
- removed link base_link
- removed link left_finger
- removed link link6
- removed link right_finger
- added link base, mass 0.873654; visual mesh filename=base.stl scale=1 1 1
- added link gripper, mass 0.553219; visual mesh filename=gripper.stl scale=1 1 1
- added link tip_left, mass 0.069657; visual mesh filename=tip_left.stl scale=1 1 1
- added link tip_right, mass 0.069657; visual mesh filename=tip_right.stl scale=1 1 1
- link link1: mass None -> 0.101218; geometry visual mesh filename=link1.stl scale=1 1 1
- link link2: mass None -> 1.46908; geometry visual mesh filename=link2.stl scale=1 1 1
- link link3: mass None -> 0.982553; geometry visual mesh filename=link3.stl scale=1 1 1
- link link4: mass None -> 0.462165; geometry visual mesh filename=link4.stl scale=1 1 1
- link link5: mass None -> 0.403307; geometry visual mesh filename=link5.stl scale=1 1 1
Joints:
- removed joint left_finger_joint
- removed joint right_finger_joint
- added joint joint7: type prismatic, parent gripper, child tip_left, origin xyz=-0.0239931 0.0445119 -0.0566829 rpy=1.02229e-14 4.71845e-16 1.68314e-15, axis 6.86541e-15 1 0, limit lower=-0.04695 upper=4.60927e-15 effort=1 velocity=1
- added joint joint8: type prismatic, parent gripper, child tip_right, origin xyz=0.0239931 -0.0445119 -0.0566829 rpy=9.6084e-15 -2.77556e-16 -3.77189e-15, axis -6.86541e-15 -1 0, limit lower=-0.04695 upper=0 effort=1 velocity=1
- joint joint1: axis 0 0 1 -> -1 0 0; limit lower=-3.14 upper=3.14 effort=1 velocity=1 -> lower=-2.61799 upper=3.14159 effort=1 velocity=1; origin xyz=0 0 0.04 rpy=0 0 0 -> xyz=-2.49777947129965e-07 -9.17402363407408e-13 0.0679999999995413 rpy=0 1.5708 3.1415963267949; parent base_link -> base
- joint joint2: axis 0 1 0 -> 3.58252e-15 1 -3.2007e-16; limit lower=-3.14 upper=3.14 effort=1 velocity=1 -> lower=-8.88178e-16 upper=3.66519 effort=1 velocity=1; origin xyz=0 0 0.08 rpy=0 0 0 -> xyz=-0.0455 -0.0339 -0.02 rpy=-1.7953e-16 5.55112e-17 -3.14159
- joint joint3: axis 0 1 0 -> 4.54273e-15 1 1.04275e-14; limit lower=-3.14 upper=3.14 effort=1 velocity=1 -> lower=0 upper=3.14159 effort=1 velocity=1; origin xyz=0 0 0.24 rpy=0 0 0 -> xyz=4.08431e-07 -0.0688 0.264 rpy=-2.99502e-14 -1.6015e-14 -3.14159
- joint joint4: axis 1 0 0 -> 0 1 0; limit lower=-3.14 upper=3.14 effort=1 velocity=1 -> lower=-1.69297 upper=1.5708 effort=1 velocity=1; origin xyz=0 0 0.24 rpy=0 0 0 -> xyz=-0.0600003 -0.0688 -0.244999 rpy=2.95536e-14 8.52374e-14 -2.10585e-14
- joint joint5: axis 0 1 0 -> 1 0 0; limit lower=-3.14 upper=3.14 effort=1 velocity=1 -> lower=-1.5708 upper=1.5708 effort=1 velocity=1; origin xyz=0 0 0.10 rpy=0 0 0 -> xyz=-0.0405003 0.0338995 -0.0739989 rpy=2.73264e-14 -4.32956e-16 -8.32667e-17
- joint joint6: axis 1 0 0 -> 1.46014e-15 2.40808e-14 -1; child link6 -> gripper; limit lower=-3.14 upper=3.14 effort=1 velocity=1 -> lower=-2.0944 upper=2.0944 effort=1 velocity=1; origin xyz=0 0 0.10 rpy=0 0 0 -> xyz=0.0404996 2.39858e-07 -0.0356 rpy=8.83309e-16 -5.88588e-16 7.69861e-14
