Commit message: Simplify evaluation presets and retain explicit TCP support

File: src/robots/zoo/agilex_piper/assets/piper_description/urdf/piper_description.urdf (robot description, URDF)
Before this commit: robot piper, 11 links, 10 joints
Links:
- added link tcp
Joints:
- added joint eef_to_tcp: type fixed, parent gripper_base, child tcp, origin xyz=0 0 0.1348875 rpy=0 0 0

File: src/robots/zoo/arx_x5/assets/X5A/urdf/X5A.urdf (robot description, URDF)
Before this commit: robot X5A, 9 links, 8 joints
Links:
- added link tcp
Joints:
- added joint eef_to_tcp: type fixed, parent link6, child tcp, origin xyz=0.1566575 0 -0.00014 rpy=0 1.570796327 0

File: src/robots/zoo/dual_yam/assets/yam.urdf (robot description, URDF)
Before this commit: robot yam, 9 links, 8 joints
Links:
- added link tcp
Joints:
- added joint eef_to_tcp: type fixed, parent gripper, child tcp, origin xyz=0 0 -0.14593 rpy=3.141592654 0 0
